Commit message: fix robot navigation inprogress

File: rb_description/urdf/robot.xacro (robot description, xacro)
@@ -35,6 +35,6 @@
         visualize_ray="false"
     />
-    <xacro:m_camera
-    />
+    <!-- <xacro:m_camera
+    /> -->
     <!-- define controller (differential drive controller) -->
     <gazebo>

File: rb_description/urdf/wheel.xacro (robot description, xacro)
@@ -8,5 +8,5 @@
             <parent link="${WHEEL_PARENT}" />
             <axis xyz="0 0 1" rpy="0 0 0" />
-            <limit effort="10000" velocity="1000" />
+            <limit effort="1000" velocity="1000" />
             <joint_properties damping="${RB_WHEEL_DAMP}" friction="${RB_WHEEL_FRICTION}" />
         </joint>

Commit message: update costmap param

File: rb_description/urdf/robot.xacro (robot description, xacro)
@@ -3,6 +3,4 @@
     <!-- define robot property -->
     <xacro:property name="PI" value="3.14159265"/>
-    <!-- <xacro:property name="rb_wheel_offx" value="40e-3"/>
-    <xacro:property name="rb_wheel_offy" value="65e-3"/> -->
     <xacro:property name="RB_H" value="45e-3"/>
     <xacro:property name="RB_BWHEEL_OFFX" value="170e-3"/>
@@ -35,6 +33,5 @@
         visualize_ray="false"
     />
-    <!-- <xacro:m_camera
-    /> -->
+    <xacro:m_camera/>
     <!-- define controller (differential drive controller) -->
     <gazebo>
@@ -43,5 +40,5 @@
             <legacyMode>false</legacyMode>
             <alwaysOn>true</alwaysOn>
-            <updateRate>50</updateRate>
+            <updateRate>100</updateRate>
             <leftJoint>left_wheel_joint</leftJoint>
             <rightJoint>right_wheel_joint</rightJoint>
@@ -53,4 +50,7 @@
             <odometryFrame>odom</odometryFrame>
             <robotBaseFrame>base_footprint</robotBaseFrame>
+            <publishWheelTF>false </publishWheelTF>
+            <publishOdomTF>true</publishOdomTF>
+            <publishWheelJointState>false</publishWheelJointState>
         </plugin>
     </gazebo>
